Commit message: added more xacro files

File: src/yardguard_description/urdf/output/yardguard.urdf (robot description, URDF)
Before this commit: robot yardguard, 7 links, 6 joints
Links:
- link back_left_wheel: geometry visual cylinder length=0.05 radius=0.1
- link back_right_wheel: geometry visual cylinder length=0.05 radius=0.1
- link front_left_wheel: geometry visual cylinder length=0.05 radius=0.1
- link front_right_wheel: geometry visual cylinder length=0.05 radius=0.1

File: src/yardguard_description/urdf/yardguard.xacro (robot description, xacro)
@@ -1,8 +1,11 @@
 <?xml version="1.0" ?>
-<!-- =================================================================================== -->
-<!-- |    This document was autogenerated by xacro from /home/daniel/projects/yard_guard/src/yardguard_description/urdf/yardguard.urdf | -->
-<!-- |    EDITING THIS FILE BY HAND IS NOT RECOMMENDED                                 | -->
-<!-- =================================================================================== -->
-<robot name="yardguard">
+<robot name="yardguard" xmlns:xacro="http://www.ros.org/wiki/xacro">
+  <xacro:include filename="mobile_base_gazebo.xacro" />
+  <!-- <xacro:include filename="common_properties.xacro" /> -->
+  <xacro:property name="base_length" value="0.288" />
+  <xacro:property name="base_width" value="0.24" />
+  <xacro:property name="base_height" value="0.1" />
+  <xacro:property name="wheel_radius" value="0.1" />
+  <xacro:property name="wheel_length" value="0.05" />
   <material name="grey">
     <color rgba="0.5 0.5 0.5 1"/>
@@ -22,5 +25,5 @@
     <visual>
       <geometry>
-        <box size="0.288 0.24 0.1"/>
+        <box size="${base_length} ${base_width} ${base_height} "/>
       </geometry>
       <origin rpy="0 0 0" xyz="0 0 0"/>
@@ -52,5 +55,5 @@
     <visual>
       <geometry>
-        <cylinder length="0.055" radius="0.07"/>
+        <cylinder length="${wheel_length}" radius="${wheel_radius}"/>
       </geometry>
       <origin rpy="1.57 0 0" xyz="0 0 0"/>
@@ -67,5 +70,5 @@
     <visual>
       <geometry>
-        <cylinder length="0.055" radius="0.07"/>
+        <cylinder length="${wheel_length}" radius="${wheel_radius}"/>
       </geometry>
       <origin rpy="1.57 0 0" xyz="0 0 0"/>
@@ -82,5 +85,5 @@
     <visual>
       <geometry>
-        <cylinder length="0.055" radius="0.07"/>
+        <cylinder length="${wheel_length}" radius="${wheel_radius}"/>
       </geometry>
       <origin rpy="1.57 0 0" xyz="0 0 0"/>
@@ -97,5 +100,5 @@
     <visual>
       <geometry>
-        <cylinder length="0.055" radius="0.07"/>
+        <cylinder length="${wheel_length}" radius="${wheel_radius}"/>
       </geometry>
       <origin rpy="1.57 0 0" xyz="0 0 0"/>
