Commit message: Added some changes

File: src/yardguard_description/urdf/mobile_base.xacro (robot description, xacro)
@@ -11,5 +11,5 @@
     <parent link="base_footprint"/>
     <child link="base_link"/>
-    <origin rpy="0 0 0" xyz="0 0 0.1"/>
+    <origin rpy="0 0 0" xyz="0 0 ${wheel_radius + 0.037}"/>
   </joint>
   <!-- base_link and base_scan (required for Nav2) -->

File: src/yardguard_description/urdf/mobile_base_gazebo.xacro (robot description, xacro)
@@ -11,4 +11,6 @@
             <left_joint>back_left_wheel_joint</left_joint>
             <right_joint>back_right_wheel_joint</right_joint>
+            <left_joint>front_left_wheel_joint</left_joint>
+            <right_joint>front_right_wheel_joint</right_joint>
             <wheel_separation>0.45</wheel_separation>
             <wheel_radius>0.1</wheel_radius>
@@ -23,4 +25,6 @@
             <joint_name>back_left_wheel_joint</joint_name>
             <joint_name>back_right_wheel_joint</joint_name>
+            <joint_name>front_left_wheel_joint</joint_name>
+            <joint_name>front_right_wheel_joint</joint_name>
         </plugin>
     </gazebo>

File: src/yardguard_description/urdf/output/yardguard.urdf (robot description, URDF)
Before this commit: robot yardguard, 7 links, 6 joints
Joints:
- joint base_joint: origin xyz=0 0 0.1 rpy=0 0 0 -> xyz=0 0 0.137 rpy=0 0 0

Commit message: added camera sensor

File: src/yardguard_description/urdf/mobile_base.xacro (robot description, xacro)
@@ -3,5 +3,5 @@
   <xacro:property name="base_length" value="0.288" />
   <xacro:property name="base_width" value="0.24" />
-  <xacro:property name="base_height" value="0.1" />
+  <xacro:property name="base_height" value="0.15" />
   <xacro:property name="wheel_radius" value="0.1" />
   <xacro:property name="wheel_length" value="0.05" />

File: src/yardguard_description/urdf/output/yardguard.urdf (robot description, URDF)
Before this commit: robot yardguard, 7 links, 6 joints
Links:
- added link camera_link, mass 0.1; collision box size=0.01 0.05 0.05; visual box size=0.01 0.05 0.05
- added link camera_link_optical
- link base_link: geometry collision box size=0.288 0.24 0.15; visual box size=0.288 0.24 0.15
Joints:
- added joint base_camera_joint: type fixed, parent base_link, child camera_link, origin xyz=0.149 0 0.0375 rpy=0 0 0
- added joint camera_optical_joint: type fixed, parent camera_link, child camera_link_optical, origin xyz=0 0 0 rpy=-1.5707963267948966 0 -1.5707963267948966

File: src/yardguard_description/urdf/yardguard.xacro (robot description, xacro)
@@ -4,3 +4,4 @@
   <xacro:include filename="mobile_base.xacro" />
   <xacro:include filename="mobile_base_gazebo.xacro" />
+  <xacro:include filename="camera.xacro" />
 </robot>
